File: pcb/fg06-c3dev-revb/fg06-c3dev-revb.kicad_sch (KiCad schematic)
At the start: 13 parts, among them J1 Conn_01x12, SW1 SW_Push, SW2 SW_DIP_x01, U1 AE-USB2.0-TYPE-C, U2 M5STAMP-C3, U3 KMR-1.8SPI

Commit message: fix footprint
Parts:
- U2: footprint fg-series:M5Stamp-C3 -> fg-series:M5STAMP-C3
Changed lines of the file:
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@@
     (property "Reference" "U2" (id 0) (at 55.88 30.48 0))
     (property "Value" "M5STAMP-C3" (id 1) (at 55.88 33.02 0))
-    (property "Footprint" "fg-series:M5Stamp-C3" (id 2) (at 55.88 68.58 0)
+    (property "Footprint" "fg-series:M5STAMP-C3" (id 2) (at 55.88 68.58 0)
       (effects (font (size 1.27 1.27)) hide)
     )
@@
     )
     (path "/10c48438-00f1-47d1-b485-8d08aa362ebb"
-      (reference "U2") (unit 1) (value "M5STAMP-C3") (footprint "fg-series:M5Stamp-C3")
+      (reference "U2") (unit 1) (value "M5STAMP-C3") (footprint "fg-series:M5STAMP-C3")
     )
     (path "/b757ff68-1d62-4528-8a8b-3d836512d501"

Commit message: place
Parts:
- renumbered SW2 to JP1
Changed lines of the file:
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@@
   (symbol (lib_id "Switch:SW_DIP_x01") (at 80.01 106.68 0) (unit 1)
     (in_bom yes) (on_board yes)
-    (property "Reference" "SW2" (id 0) (at 80.01 99.8982 0))
+    (property "Reference" "JP1" (id 0) (at 80.01 99.8982 0))
     (property "Value" "SW_DIP_x01" (id 1) (at 80.01 102.2096 0))
     (property "Footprint" "Connector_PinHeader_2.54mm:PinHeader_1x02_P2.54mm_Vertical" (id 2) (at 80.01 106.68 0)
@@
       (reference "J1") (unit 1) (value "Conn_01x12") (footprint "Connector_PinHeader_2.54mm:PinHeader_1x12_P2.54mm_Vertical")
     )
+    (path "/81b6f73b-0f33-482e-b717-6735907e390f"
+      (reference "JP1") (unit 1) (value "SW_DIP_x01") (footprint "Connector_PinHeader_2.54mm:PinHeader_1x02_P2.54mm_Vertical")
+    )
     (path "/2a8d72e0-d230-4a61-aa17-fadec28ff265"
       (reference "R1") (unit 1) (value "R") (footprint "Resistor_THT:R_Axial_DIN0207_L6.3mm_D2.5mm_P7.62mm_Horizontal")
@@
       (reference "SW1") (unit 1) (value "SW_Push") (footprint "Button_Switch_THT:SW_PUSH_6mm")
     )
-    (path "/81b6f73b-0f33-482e-b717-6735907e390f"
-      (reference "SW2") (unit 1) (value "SW_DIP_x01") (footprint "Connector_PinHeader_2.54mm:PinHeader_1x02_P2.54mm_Vertical")
-    )
     (path "/0fa9fc53-01f4-4a24-bd32-138cbaf08933"
