File: pcb/fg06-c3dev-revb/fg06-c3dev-revb.kicad_pcb (KiCad board)
At the start: 2 copper layers, 90 x 55 mm, 4 parts

Commit message: place
Parts:
- added J1: Conn_01x12, Connector_PinHeader_2.54mm:PinHeader_1x12_P2.54mm_Vertical, F.Cu at (117.6, 89.9)
- added JP1: SW_DIP_x01, Connector_PinHeader_2.54mm:PinHeader_1x02_P2.54mm_Vertical, F.Cu at (71.4, 79.8)
- added R1: R, Resistor_THT:R_Axial_DIN0207_L6.3mm_D2.5mm_P7.62mm_Horizontal, F.Cu at (46.7, 74.9)
- added R2: R, Resistor_THT:R_Axial_DIN0207_L6.3mm_D2.5mm_P7.62mm_Horizontal, F.Cu at (56.9, 74.9)
- added R3: R, Resistor_THT:R_Axial_DIN0207_L6.3mm_D2.5mm_P7.62mm_Horizontal, F.Cu at (68.3, 43.2)
- added R4: R, Resistor_THT:R_Axial_DIN0207_L6.3mm_D2.5mm_P7.62mm_Horizontal, F.Cu at (68.3, 47.2)
- added R5: R, Resistor_THT:R_Axial_DIN0207_L6.3mm_D2.5mm_P7.62mm_Horizontal, F.Cu at (68.3, 51.3)
- added R6: R, Resistor_THT:R_Axial_DIN0207_L6.3mm_D2.5mm_P7.62mm_Horizontal, F.Cu at (68.3, 55.4)
- added R7: R, Resistor_THT:R_Axial_DIN0207_L6.3mm_D2.5mm_P7.62mm_Horizontal, F.Cu at (68.3, 59.4)
- added SW1: SW_Push, Button_Switch_THT:SW_PUSH_6mm, F.Cu at (68.6, 84.8)
- added U1: AE-USB2.0-TYPE-C, fg-series:AE-USB2.0-TYPE-C, F.Cu at (55.3, 86.2)
- added U2: M5STAMP-C3, fg-series:M5STAMP-C3, F.Cu at (55.6, 54.6)
- added U3: KMR-1.8SPI, fg-series:KMR-1.8SPI, F.Cu at (104.5, 64.8)
- moved REF3 0.05 mm to (124.0, 44.7)
Other:
- board text added: "1"
- board text added: "12"
- board text added: "12 Vcc(3.3V) 11 GND 10 G20(RX0) 09 G21(TX0) 08 G4(SCLK) 07 G5(MOSI) 06 G6(MISO) 05 G0 04 GND 03 Vcc(5V) 02 G18(D-) 01 G19(D+)"
- board text added: "AE-USB2.0-TYPE-C"
- board text added: "G1(SD_CS) G7(LCD_CS) G8(LCD_RESET) G9(SW1) G10(LCD_A0)"
- board text added: "KMR-1.8SPI"
- board text added: "M5STAMP-C3"

Commit message: fix
Routing:
- net GPIO19(D+): track 0.00 -> 106.8 mm
- net GPIO18(D-): track 0.00 -> 99.7 mm
- net Vcc_USB_5V: track 0.00 -> 93.6 mm
- net Vcc: track 0.00 -> 93.4 mm
- net MOSI: track 0.00 -> 86.9 mm
- net MISO: track 0.00 -> 75.9 mm
- net SCLK: track 0.00 -> 72.4 mm
- net GPIO0: track 0.00 -> 68.9 mm
- net GND: track 0.00 -> 65.0 mm, vias 0 -> 3
- net GPIO21(TX0): track 0.00 -> 63.7 mm
- net GPIO20(RX0): track 0.00 -> 62.5 mm
- net BOOT_SW: track 0.00 -> 52.8 mm
- net SD_CS: track 0.00 -> 32.4 mm
- net LCD_RST: track 0.00 -> 22.9 mm
- net LCD_DC: track 0.00 -> 22.2 mm
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- added copper zone on B.Cu, net GND

Commit message: update rev.B
Parts:
- moved JP1 0.81 mm to (70.6, 79.5), turned to 90 degrees
- moved R7 0.80 mm to (68.6, 58.7)
- moved R1 0.57 mm to (46.5, 74.4)
- moved R2 0.57 mm to (56.6, 74.4)
- moved R6 0.57 mm to (68.6, 54.9)
- moved SW1 0.39 mm to (68.8, 85.1)
- moved U2 0.37 mm to (55.4, 54.9)
- moved R3 0.36 mm to (68.6, 43.4)
- moved R5 0.36 mm to (68.6, 51.1)
- moved U1 0.27 mm to (55.1, 86.1)
- moved R4 0.25 mm to (68.6, 47.2)
- moved J1 0.25 mm to (117.9, 89.9)
Routing:
- net GPIO19(D+): track 106.8 -> 0.00 mm
- net GPIO18(D-): track 99.7 -> 0.00 mm
- net Vcc_USB_5V: track 93.6 -> 0.00 mm
- net Vcc: track 93.4 -> 0.00 mm
- net MOSI: track 86.9 -> 0.00 mm
- net MISO: track 75.9 -> 0.00 mm
- net SCLK: track 72.4 -> 0.00 mm
- net GPIO0: track 68.9 -> 0.00 mm
- net GND: track 65.0 -> 0.00 mm, vias 3 -> 0
- net GPIO21(TX0): track 63.7 -> 0.00 mm
- net GPIO20(RX0): track 62.5 -> 0.00 mm
- net BOOT_SW: track 52.8 -> 0.00 mm
- net SD_CS: track 32.4 -> 0.00 mm
- net LCD_RST: track 22.9 -> 0.00 mm
- net LCD_DC: track 22.2 -> 0.00 mm
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- removed copper zone on B.Cu, net GND
Other:
- board text added: "EXT_5V"
- board text added: "SW1"

Commit message: update pcb
Routing:
- net GPIO19(D+): track 0.00 -> 106.4 mm
- net Vcc: track 0.00 -> 98.6 mm
- net GPIO18(D-): track 0.00 -> 97.4 mm
- net Vcc_USB_5V: track 0.00 -> 91.1 mm
- net MOSI: track 0.00 -> 84.1 mm
- net MISO: track 0.00 -> 76.6 mm
- net SCLK: track 0.00 -> 72.8 mm
- net GPIO20(RX0): track 0.00 -> 70.5 mm
- net GPIO0: track 0.00 -> 70.2 mm
- net GPIO21(TX0): track 0.00 -> 68.9 mm
- net BOOT_SW: track 0.00 -> 52.0 mm
- net SD_CS: track 0.00 -> 29.9 mm
- net LCD_RST: track 0.00 -> 28.1 mm
- net LCD_DC: track 0.00 -> 27.0 mm
- net LCD_CS: track 0.00 -> 21.8 mm
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- added copper zone on B.Cu, net GND
- added copper zone on F.Cu, net GND
